File: Hardware/ESP32-cnc/_autosave-ESP32-cnc.kicad_pcb (KiCad board)
At the start: 2 copper layers, 100 x 100 mm, 85 parts, among them J1 Inputs, J10 Y-Servo, J11 X_STEP_B, J12 Y_STEP_B, J13 Spindle On/Off, J14 X_STEP_A, J15 Y_STEP_A, J16 Z_STEP, J2 12-18V DC, J3 Conn_01x19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

Commit message: minor updates
Other:
- board text added: "+5V"
- board text added: "EPS32-GRBL-CNC V1.0 CC BY 3.0"
- board text added: "GND"
- board text added: "ILCK"
- board text added: "PWM"
- board text added: "SPINDLE 5V PWM"
- board text removed: "PWM SPINDLE 5V"
Changed lines of the file:
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@@
   (general
     (thickness 1.6)
-    (drawings 26)
+    (drawings 39)
     (tracks 724)
     (zones 0)
@@
     (descr "Through hole straight pin header, 2x05, 2.54mm pitch, double rows")
     (tags "Through hole pin header THT 2x05 2.54mm double row")
-    (fp_text reference J7 (at 1.27 -2.33) (layer F.SilkS)
+    (fp_text reference J7 (at 2.9845 -2.6035) (layer F.SilkS)
       (effects (font (size 1 1) (thickness 0.15)))
     )
@@
     (descr "Through hole straight pin header, 1x02, 2.54mm pitch, single row")
     (tags "Through hole pin header THT 1x02 2.54mm single row")
-    (fp_text reference J5 (at -0.1425 6.3425 180) (layer F.SilkS)
+    (fp_text reference J5 (at 1.7145 5.461 180) (layer F.SilkS)
       (effects (font (size 1 1) (thickness 0.15)))
     )
@@
       (net 2 GND))
   )
+  (gr_text GND (at 103.505 87.884 90) (layer F.SilkS)
+    (effects (font (size 1 1) (thickness 0.15)))
+  )
+  (gr_text PWM (at 101.0285 87.884 90) (layer F.SilkS)
+    (effects (font (size 1 1) (thickness 0.15)))
+  )
+  (gr_text ILCK (at 97.028 88.773) (layer F.SilkS)
+    (effects (font (size 1 1) (thickness 0.15)))
+  )
+  (gr_text GND (at 105.4735 83.312 90) (layer F.SilkS)
+    (effects (font (size 1 1) (thickness 0.15)))
+  )
+  (gr_text GND (at 107.315 48.26) (layer F.SilkS)
+    (effects (font (size 1 1) (thickness 0.15)))
+  )
+  (gr_text GND (at 107.315 53.213) (layer F.SilkS)
+    (effects (font (size 1 1) (thickness 0.15)))
+  )
+  (gr_text GND (at 107.315 58.3565) (layer F.SilkS)
+    (effects (font (size 1 1) (thickness 0.15)))
+  )
+  (gr_text "GND\n" (at 107.315 63.4365) (layer F.SilkS)
+    (effects (font (size 1 1) (thickness 0.15)))
+  )
+  (gr_text GND (at 105.664 66.4845 90) (layer F.SilkS)
+    (effects (font (size 1 1) (thickness 0.15)))
+  )
+  (gr_text +5V (at 73.4695 120.777 90) (layer F.SilkS)
+    (effects (font (size 1 1) (thickness 0.15)))
+  )
+  (gr_text GND (at 70.866 120.5865 90) (layer F.SilkS)
+    (effects (font (size 1 1) (thickness 0.15)))
+  )
+  (gr_text GND (at 51.689 132.08 90) (layer F.SilkS)
+    (effects (font (size 1 1) (thickness 0.15)))
+  )
+  (gr_text "EPS32-GRBL-CNC\nV1.0\nCC BY 3.0" (at 76.5175 129.032) (layer F.SilkS)
+    (effects (font (size 1 1) (thickness 0.25)))
+  )
   (gr_text "X-AXIS 2" (at 16.637 50.292 90) (layer F.SilkS)
     (effects (font (size 1 1) (thickness 0.15)))
@@
     (effects (font (size 1 1) (thickness 0.15)))
   )
-  (gr_text "PROBE\n" (at 108.2675 60.96) (layer F.SilkS)
+  (gr_text "PROBE\n" (at 108.267381 60.96) (layer F.SilkS)
     (effects (font (size 1 1) (thickness 0.15)))
   )
-  (gr_text RESET (at 108.0135 55.88) (layer F.SilkS)
+  (gr_text RESET (at 108.053096 55.88) (layer F.SilkS)
     (effects (font (size 1 1) (thickness 0.15)))
   )
-  (gr_text START (at 107.823 50.927) (layer F.SilkS)
+  (gr_text START (at 107.957857 50.927) (layer F.SilkS)
     (effects (font (size 1 1) (thickness 0.15)))
   )
-  (gr_text HOLD (at 107.3785 45.6565) (layer F.SilkS)
+  (gr_text HOLD (at 107.743572 45.6565) (layer F.SilkS)
     (effects (font (size 1 1) (thickness 0.15)))
   )
@@
     (effects (font (size 1 1) (thickness 0.15)))
   )
-  (gr_text "PWM SPINDLE 5V" (at 99.8855 88.392) (layer F.SilkS)
+  (gr_text "SPINDLE\n5V PWM" (at 108.331 90.7415 90) (layer F.SilkS)
     (effects (font (size 1 1) (thickness 0.15)))
   )
-  (gr_text X (at 108.5215 69.5325 90) (layer F.SilkS)
+  (gr_text X (at 108.458 69.5325 90) (layer F.SilkS)
     (effects (font (size 1 1) (thickness 0.15)))
   )
-  (gr_text X (at 108.5215 72.0725 90) (layer F.SilkS)
+  (gr_text X (at 108.458 72.0725 90) (layer F.SilkS)
     (effects (font (size 1 1) (thickness 0.15)))
   )
-  (gr_text Y (at 108.3945 74.676 90) (layer F.SilkS)
+  (gr_text Y (at 108.458 74.676 90) (layer F.SilkS)
     (effects (font (size 1 1) (thickness 0.15)))
   )
@@
     (effects (font (size 1 1) (thickness 0.15)))
   )
-  (gr_text FAN (at 72.0725 127) (layer F.SilkS)
+  (gr_text FAN (at 77.0255 124.0155) (layer F.SilkS)
     (effects (font (size 1 1) (thickness 0.15)))
   )
